File: Hardware/Linear_PowerSup_v1.kicad_pcb (KiCad board)
At the start: 2 copper layers, 105 x 105 mm, 13 parts, among them J1 Conn_01x02, J2 Conn_01x02, U1 TSR3-2450N

Commit message: Add files via upload
Routing:
- net GND: track 90.4 -> 0.00 mm
- net Net-(U1-Vout): track 26.7 -> 28.3 mm
- net Net-(D1-Pad2): track 21.7 -> 20.9 mm
- net Net-(D2-A): track 8.43 -> 7.93 mm
- added copper zone on B.Cu, net GND
- added copper zone on F.Cu, net GND
Changed lines of the file:
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@@
+	)
+	(segment
+		(start 91 110.5)
+		(end 96 105.5)
+		(width 1.5)
+		(layer "F.Cu")
+		(net 1)
+	)
+	(segment
+		(start 95.1 93.1)
+		(end 96 94)
+		(width 1.5)
+		(layer "F.Cu")
+		(net 1)
+	)
+	(segment
+		(start 101.34 79.76)
+		(end 95.1 86)
+		(width 1.5)
+		(layer "F.Cu")
+		(net 1)
 	)
 	(segment
@@
 	)
 	(segment
-		(start 96.76 86)
-		(end 103 79.76)
+		(start 103 79.76)
+		(end 101.34 79.76)
 		(width 1.5)
 		(layer "F.Cu")
@@
 	(segment
 		(start 96 105.5)
-		(end 91 110.5)
-		(width 1.5)
-		(layer "F.Cu")
-		(net 1)
-	)
-	(segment
-		(start 95.1 86)
-		(end 96.76 86)
-		(width 1.5)
-		(layer "F.Cu")
-		(net 1)
-	)
-	(segment
-		(start 95.1 93.1)
 		(end 96 94)
 		(width 1.5)
@@
 	)
 	(segment
-		(start 96 94)
-		(end 96 105.5)
-		(width 1.5)
-		(layer "F.Cu")
-		(net 1)
-	)
-	(segment
-		(start 93.5 69.5)
-		(end 96 72)
-		(width 1.5)
-		(layer "F.Cu")
-		(net 2)
-	)
-	(segment
-		(start 92.5 68.5)
-		(end 93.5 69.5)
-		(width 1.5)
-		(layer "F.Cu")
-		(net 2)
-	)
-	(segment
-		(start 82 94)
-		(end 80 92)
-		(width 1.5)
-		(layer "F.Cu")
-		(net 2)
-	)
-	(segment
-		(start 81.7977 68.5)
-		(end 92.5 68.5)
-		(width 1.5)
-		(layer "F.Cu")
-		(net 2)
-	)
-	(segment
-		(start 94.299 97.299)
-		(end 94.299 104.201)
-		(width 1.5)
-		(layer "F.Cu")
-		(net 2)
-	)
-	(segment
-		(start 91 94)
-		(end 82 94)
-		(width 1.5)
-		(layer "F.Cu")
-		(net 2)
-	)
-	(segment
-		(start 96 72)
-		(end 96 80)
-		(width 1.5)
-		(layer "F.Cu")
-		(net 2)
-	)
-	(segment
-		(start 88 110.5)
-		(end 83.5 110.5)
-		(width 1.5)
-		(layer "F.Cu")
-		(net 2)
-	)
-	(segment
-		(start 94.299 104.201)
-		(end 88 110.5)
-		(width 1.5)
-		(layer "F.Cu")
-		(net 2)
-	)
-	(segment
-		(start 91 94)
-		(end 94.299 97.299)
-		(width 1.5)
-		(layer "F.Cu")
-		(net 2)
-	)
-	(segment
-		(start 93.4 86)
-		(end 93.4 91.6)
-		(width 1.5)
-		(layer "B.Cu")
-		(net 2)
-	)
-	(segment
-		(start 93.4 82.6)
-		(end 96 80)
-		(width 1.5)
-		(layer "B.Cu")
-		(net 2)
-	)
-	(segment
-		(start 93.4 91.6)
-		(end 91 94)
-		(width 1.5)
-		(layer "B.Cu")
-		(net 2)
-	)
-	(segment
-		(start 103 95)
-		(end 100.249 92.249)
-		(width 1.5)
-		(layer "B.Cu")
-		(net 2)
-	)
-	(segment
-		(start 92.751 92.249)
-		(end 91 94)
-		(width 1.5)
-		(layer "B.Cu")
-		(net 2)
-	)
-	(segment
-		(start 100.249 92.249)
-		(end 92.751 92.249)
-		(width 1.5)
-		(layer "B.Cu")
-		(net 2)
-	)
-	(segment
-		(start 93.4 86)
-		(end 93.4 82.6)
-		(width 1.5)
-		(layer "B.Cu")
-		(net 2)
+		(start 91 75.5)
+		(end 93.5 73)
+		(width 0.2)
+		(layer "F.Cu")
+		(net 3)
+	)
+	(segment
+		(start 91 80)
+		(end 91 75.5)
+		(width 0.2)
+		(layer "F.Cu")
+		(net 3)
+	)
+	(segment
+		(start 83 80.01)
+		(end 86 77.01)
+		(width 0.2)
+		(layer "F.Cu")
+		(net 3)
+	)
+	(segment
+		(start 91 80)
+		(end 91 81)
+		(width 0.2)
+		(layer "F.Cu")
+		(net 3)
+	)
+	(segment
+		(start 91.7 81.7)
+		(end 91.7 86)
+		(width 0.2)
+		(layer "F.Cu")
+		(net 3)
 	)
 	(segment
@@
 	)
 	(segment
-		(start 91 76)
+		(start 88.99 80)
 		(end 91 80)
 		(width 0.2)
@@
 	)
 	(segment
-		(start 83 80.01)
-		(end 86 77.01)
-		(width 0.2)
-		(layer "F.Cu")
-		(net 3)
-	)
-	(segment
-		(start 87.5 74.5)
-		(end 89 76)
-		(width 0.2)
-		(layer "F.Cu")
-		(net 3)
-	)
-	(segment
-		(start 93.5 73.5)
-		(end 91 76)
-		(width 0.2)
-		(layer "F.Cu")
-		(net 3)
-	)
-	(segment
-		(start 86 74.5)
-		(end 87.5 74.5)
-		(width 0.2)
-		(layer "F.Cu")
-		(net 3)
-	)
-	(segment
-		(start 89 76)
-		(end 91 76)
-		(width 0.2)
-		(layer "F.Cu")
-		(net 3)
-	)
-	(segment
-		(start 91 80.5)
-		(end 91.7 81.2)
-		(width 0.2)
-		(layer "B.Cu")
+		(start 91 81)
+		(end 91.7 81.7)
+		(width 0.2)
+		(layer "F.Cu")
+		(net 3)
+	)
+	(segment
+		(start 86 77.01)
+		(end 88.99 80)
+		(width 0.2)
+		(layer "F.Cu")
 		(net 3)
 	)
@@
 	)
 	(segment
-		(start 91.7 81.2)
-		(end 91.7 86)
-		(width 0.2)
-		(layer "B.Cu")
-		(net 3)
+		(start 164 92)
+		(end 164 94.490575)
+		(width 1)
+		(layer "F.Cu")
+		(net 4)
 	)
 	(segment
@@
 	)
 	(segment
-		(start 148.490165 110.00041)
-		(end 164 94.490575)
-		(width 1)
-		(layer "B.Cu")
+		(start 164 94.490575)
+		(end 148.490165 110.00041)
+		(width 1)
+		(layer "F.Cu")
 		(net 4)
 	)
 	(segment
-		(start 164 94.490575)
-		(end 164 92)
-		(width 1)
-		(layer "B.Cu")
-		(net 4)
+		(start 118 104.15)
+		(end 103.77 89.92)
+		(width 1.5)
+		(layer "F.Cu")
+		(net 5)
 	)
 	(segment
@@
 	)
 	(segment
-		(start 103 89.92)
-		(end 117.23 104.15)
-		(width 1.5)
-		(layer "B.Cu")
-		(net 5)
-	)
-	(segment
-		(start 117.23 104.15)
-		(end 118 104.15)
-		(width 1.5)
-		(layer "B.Cu")
-		(net 5)
-	)
-	(segment
-		(start 79.2577 70.3377)
-		(end 74.5954 75)
+		(start 74.5954 74.5)
+		(end 79.2577 69.8377)
 		(width 0.2)
 		(layer "F.Cu")
@@
 	)
 	(segment
-		(start 79.2577 68.5)
-		(end 79.2577 70.3377)
+		(start 79.2577 69.8377)
+		(end 79.2577 68.5)
 		(width 0.2)
 		(layer "F.Cu")
 		(net 6)
+	)
+	(segment
+		(start 164 75)
+		(end 163 74)
+		(width 1)
+		(layer "F.Cu")
+		(net 7)
 	)
 	(segment
@@
 		(end 164 75)
 		(width 1)
-		(layer "B.Cu")
+		(layer "F.Cu")
 		(net 7)
 	)
 	(segment
-		(start 164 75)
-		(end 163 74)
-		(width 1)
-		(layer "B.Cu")
-		(net 7)
-	)
-	(segment
-		(start 77.92 80)
+		(start 80 82.08)
+		(end 77.92 80)
+		(width 0.2)
+		(layer "F.Cu")
+		(net 8)
+	)
+	(segment
+		(start 80 87)
 		(end 80 82.08)
 		(width 0.2)
@@
 	)
 	(segment
-		(start 80 82.08)
-		(end 80 87)
-		(width 0.2)
-		(layer "F.Cu")
-		(net 8)
+		(start 118 80.83)
+		(end 107.01 80.83)
+		(width 1.5)
+		(layer "F.Cu")
+		(net 9)
 	)
 	(segment
@@
 		(end 103 84.84)
 		(width 1.5)
-		(layer "B.Cu")
-		(net 9)
-	)
-	(segment
-		(start 118 80.83)
-		(end 107.01 80.83)
-		(width 1.5)
-		(layer "B.Cu")
+		(layer "F.Cu")
 		(net 9)
 	)
@@
 		(end 148.459835 74.99959)
 		(width 1)
-		(layer "B.Cu")
+		(layer "F.Cu")
 		(net 10)
 	)
@@
 		(end 154.539425 68.92)
 		(width 1)
-		(layer "B.Cu")
+		(layer "F.Cu")
 		(net 10)
 	)
+	(zone
+		(net 2)
+		(net_name "GND")
+		(layers "F.Cu" "B.Cu")
+		(hatch edge 0.5)
+		(connect_pads
+			(clearance 0.5)
+		)
+		(min_thickness 0.25)
+		(filled_areas_thickness no)
+		(fill yes
+			(thermal_gap 0.5)
+			(thermal_bridge_width 0.5)
+		)
+		(polygon
+			(pts
+				(xy 65.5 35.5) (xy 179 34.5) (xy 179.5 148.5) (xy 62 147.5)
+			)
+		)
+	)
 	(embedded_fonts no)
